File: kicad/diamond.kicad_pcb (KiCad board)
At the start: 2 copper layers, 76.5 x 66.3 mm, 40 parts, among them J1 INPUT, Q1 BD139, Q2 BD140, Q3 NJW0281G, Q4 NJW0302G, U1 NE5532

Commit message: Cleanup
Parts:
- moved R3 14.8 mm to (102.1, 94.2)
- moved D1 10.5 mm to (112.3, 105.4)
- moved C1 9.86 mm to (102.8, 101.3)
Connections:
- U1 pad 5: Net-(U1B-+) -> GND
- U1 pad 6: Net-(U1B-+) -> Net-(U1B--)
- U1 pad 7: Net-(U1B-+) -> Net-(U1B--)
Routing:
- net Net-(U1A--): track 42.9 -> 26.4 mm
- net GND: track 120.2 -> 125.6 mm
- net Net-(U1B-+): track 5.08 -> 0.00 mm
- net Net-(U1B--): track 0.00 -> 2.54 mm
- net Net-(R7-Pad2): track 42.0 -> 43.4 mm
- net Net-(D1-K): track 19.3 -> 18.6 mm
- net Net-(Q4-B): track 70.0 -> 69.5 mm
Changed lines of the file:
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@@
 	(net 14 "SPK")
 	(net 15 "Net-(R7-Pad2)")
-	(net 16 "Net-(U1B-+)")
+	(net 16 "Net-(U1B--)")
 	(net 17 "B+")
 	(net 18 "B-")
@@
 	(footprint "Resistor_THT:R_Axial_DIN0204_L3.6mm_D1.6mm_P7.62mm_Horizontal"
 		(layer "F.Cu")
-		(at 106.934 108.204 90)
+		(at 102.108 94.234 90)
 		(descr "Resistor, Axial_DIN0204 series, Axial, Horizontal, pin pitch=7.62mm, 0.167W, length*diameter=3.6*1.6mm^2, http://cdn-reichelt.de/documents/datenblatt/B400/1_4W%23YAG.pdf")
 		(tags "Resistor Axial_DIN0204 series Axial Horizontal pin pitch 7.62mm 0.167W length 3.6mm diameter 1.6mm")
@@
 			(layers "*.Cu" "*.Mask")
 			(remove_unused_layers no)
-			(net 16 "Net-(U1B-+)")
+			(net 2 "GND")
 			(pinfunction "+")
 			(pintype "input")
@@
 			(layers "*.Cu" "*.Mask")
 			(remove_unused_layers no)
-			(net 16 "Net-(U1B-+)")
+			(net 16 "Net-(U1B--)")
 			(pinfunction "-")
 			(pintype "input")
@@
 			(layers "*.Cu" "*.Mask")
 			(remove_unused_layers no)
-			(net 16 "Net-(U1B-+)")
+			(net 16 "Net-(U1B--)")
 			(pintype "output")
 		)
@@
 	(footprint "Diode_THT:D_DO-35_SOD27_P7.62mm_Horizontal"
 		(layer "F.Cu")
-		(at 122.174 108.966 90)
+		(at 112.268 105.41 90)
 		(descr "Diode, DO-35_SOD27 series, Axial, Horizontal, pin pitch=7.62mm, , length*diameter=4*2mm^2, , http://www.diodes.com/_files/packages/DO-35.pdf")
 		(tags "Diode DO-35_SOD27 series Axial Horizontal pin pitch 7.62mm  length 4mm diameter 2mm")
@@
 	(footprint "Capacitor_THT:CP_Radial_D8.0mm_P5.00mm"
 		(layer "F.Cu")
-		(at 112.348 103.632)
+		(at 102.753349 101.346)
 		(descr "CP, Radial series, Radial, pin pitch=5.00mm, , diameter=8mm, Electrolytic Capacitor")
 		(tags "CP Radial series Radial pin pitch 5.00mm  diameter 8mm Electrolytic Capacitor")
@@
 	)
 	(segment
-		(start 117.682 108.966)
-		(end 112.348 103.632)
+		(start 102.108 100.700651)
+		(end 102.753349 101.346)
 		(width 1)
 		(layer "B.Cu")
@@
 	)
 	(segment
-		(start 122.174 108.966)
-		(end 117.682 108.966)
+		(start 106.817349 105.41)
+		(end 112.268 105.41)
 		(width 1)
 		(layer "B.Cu")
@@
 	)
 	(segment
-		(start 107.776 108.204)
-		(end 112.348 103.632)
+		(start 102.108 94.234)
+		(end 102.108 100.700651)
 		(width 1)
 		(layer "B.Cu")
@@
 	)
 	(segment
-		(start 106.934 108.204)
-		(end 107.776 108.204)
+		(start 102.753349 101.346)
+		(end 106.817349 105.41)
 		(width 1)
 		(layer "B.Cu")
@@
 	)
 	(segment
+		(start 107.753349 101.346)
+		(end 108.712 101.346)
+		(width 1)
+		(layer "F.Cu")
+		(net 2)
+	)
+	(segment
+		(start 108.712 101.346)
+		(end 112.268 97.79)
+		(width 1)
+		(layer "F.Cu")
+		(net 2)
+	)
+	(segment
 		(start 134.366 97.536)
 		(end 136.652 95.25)
@@
 	)
 	(segment
+		(start 115.829 86.106)
+		(end 118.972 86.106)
+		(width 1)
+		(layer "B.Cu")
+		(net 2)
+	)
+	(segment
+		(start 118.464002 91.439998)
+		(end 125.068 84.836)
+		(width 1)
+		(layer "B.Cu")
+		(net 2)
+	)
+	(segment
 		(start 136.652 92.358304)
 		(end 129.129696 84.836)
@@
 	)
 	(segment
-		(start 117.348 92.556002)
-		(end 125.068002 84.836)
-		(width 1)
-		(layer "B.Cu")
-		(net 2)
-	)
-	(segment
 		(start 129.129696 84.836)
 		(end 125.068 84.836)
@@
 	)
 	(segment
-		(start 117.348 103.632)
-		(end 117.348 92.556002)
+		(start 118.972 86.106)
+		(end 125.068 80.01)
 		(width 1)
 		(layer "B.Cu")
@@
 	)
 	(segment
-		(start 136.652 95.25)
-		(end 136.652 101.68)
-		(width 4)
+		(start 112.268 97.79)
+		(end 118.364 97.79)
+		(width 1)
 		(layer "B.Cu")
 		(net 2)
 	)
 	(segment
-		(start 119.634 101.346)
-		(end 117.348 103.632)
-		(width 1)
+		(start 136.652 95.25)
+		(end 136.652 101.68)
+		(width 4)
 		(layer "B.Cu")
 		(net 2)
@@
 	)
 	(segment
+		(start 118.464002 91.44)
+		(end 118.464002 91.439998)
+		(width 1)
+		(layer "B.Cu")
+		(net 2)
+	)
+	(segment
 		(start 126.901674 70.005674)
 		(end 125.068002 71.839346)
@@
 	(segment
 		(start 118.464002 91.44)
-		(end 125.068002 84.836)
+		(end 114.768 91.44)
 		(width 1)
 		(layer "B.Cu")
@@
 	)
 	(segment
-		(start 114.768 91.44)
-		(end 118.464002 91.44)
-		(width 1)
-		(layer "B.Cu")
-		(net 2)
-	)
-	(segment
 		(start 136.370349 60.537)
 		(end 136.398 60.537)
@@
 	)
 	(segment
-		(start 122.174 101.346)
-		(end 119.634 101.346)
+		(start 118.364 97.79)
+		(end 124.968 91.186)
 		(width 1)
 		(layer "B.Cu")
@@
 	)
 	(segment
+		(start 103.632 82.002)
+		(end 102.108 83.526)
+		(width 1)
+		(layer "B.Cu")
+		(net 4)
+	)
+	(segment
 		(start 107.758 75.583156)
 		(end 109.71 77.535156)
@@
 	)
 	(segment
-		(start 106.934 100.584)
-		(end 105.944051 100.584)
-		(width 1)
-		(layer "B.Cu")
-		(net 4)
-	)
-	(segment
-		(start 102.231 96.870949)
-		(end 102.231 83.403)
-		(width 1)
-		(layer "B.Cu")
-		(net 4)
-	)
-	(segment
-		(start 102.231 83.403)
-		(end 103.632 82.002)
-		(width 1)
-		(layer "B.Cu")
-		(net 4)
-	)
-	(segment
-		(start 105.944051 100.584)
-		(end 102.231 96.870949)
+		(start 102.108 83.526)
+		(end 102.108 86.614)
 		(width 1)
 		(layer "B.Cu")
@@
 	)
 	(segment
-		(start 157.734 85.344)
-		(end 157.734 85.482)
+		(start 143.804 67.818)
+		(end 143.804 69.382)
 		(width 1)
 		(layer "F.Cu")
@@
 	)
 	(segment
-		(start 168.484 83.312)
-		(end 170.654 85.482)
+		(start 159.766 83.312)
+		(end 157.734 85.344)
+		(width 1)
+		(layer "F.Cu")
+		(net 12)
+	)
+	(segment
+		(start 157.734 85.344)
+		(end 157.734 85.598)
 		(width 1)
 		(layer "F.Cu")
@@
 	)
 	(segment
-		(start 144.272 67.818)
+		(start 168.484 83.312)
 		(end 159.766 83.312)
 		(width 1)
@@
 	)
 	(segment
-		(start 143.804 67.818)
-		(end 144.272 67.818)
+		(start 149.606 75.184)
+		(end 149.606 81.788)
 		(width 1)
 		(layer "F.Cu")
@@
 	)
 	(segment
-		(start 159.766 83.312)
+		(start 170.654 85.482)
 		(end 168.484 83.312)
 		(width 1)
@@
 	)
 	(segment
-		(start 157.734 85.482)
-		(end 153.532 85.482)
+		(start 157.734 85.598)
+		(end 153.416 85.598)
 		(width 1)
 		(layer "F.Cu")
@@
 	)
 	(segment
-		(start 159.766 83.312)
-		(end 157.734 85.344)
+		(start 149.606 81.788)
+		(end 153.416 85.598)
 		(width 1)
 		(layer "F.Cu")
@@
 	)
 	(segment
-		(start 153.532 85.482)
+		(start 143.804 69.382)
+		(end 149.606 75.184)
+		(width 1)
+		(layer "F.Cu")
+		(net 12)
+	)
+	(segment
+		(start 153.416 85.598)
 		(end 149.098 89.916)
 		(width 1)
@@
 	)
 	(segment
-		(start 148.59 77.216)
-		(end 142.303 70.929)
+		(start 146.170944 87.376)
+		(end 142.303 83.508056)
 		(width 1)
 		(layer "F.Cu")
@@
 	)
 	(segment
-		(start 148.285265 61.214)
-		(end 159.004 61.214)
+		(start 148.59 87.376)
+		(end 146.170944 87.376)
 		(width 1)
 		(layer "F.Cu")
@@
 	)
 	(segment
-		(start 142.303 70.929)
+		(start 142.303 83.508056)
 		(end 142.303 67.196265)
 		(width 1)
@@
 	)
 	(segment
-		(start 148.59 87.376)
-		(end 148.59 77.216)
+		(start 148.285265 61.214)
+		(end 159.004 61.214)
 		(width 1)
 		(layer "F.Cu")
@@
 	(segment
 		(start 115.829 81.026)
-		(end 115.829 86.106)
+		(end 115.829 83.566)
 		(width 1)
 		(layer "B.Cu")
@@
 	)
 	(segment
-		(start 114.046 95.718)
-		(end 114.046 103.632944)
+		(start 171.654 58.298)
+		(end 170.053 59.899)
 		(width 1)
 		(layer "B.Cu")
@@
 	)
 	(segment
-		(start 171.654 58.298)
-		(end 170.053 59.899)
+		(start 108.209 86.106)
+		(end 108.209 91.186)
 		(width 1)
 		(layer "B.Cu")
@@
 	)
 	(segment
-		(start 114.046 103.632944)
-		(end 117.093056 106.68)
+		(start 170.053 61.575)
+		(end 173.605 65.127)
 		(width 1)
 		(layer "B.Cu")
@@
 	)
 	(segment
-		(start 108.209 86.106)
-		(end 108.209 91.186)
+		(start 109.768 91.44)
+		(end 109.768 98.846)
 		(width 1)
 		(layer "B.Cu")
@@
 	)
 	(segment
-		(start 170.053 61.575)
-		(end 173.605 65.127)
+		(start 117.602 106.68)
+		(end 136.652 106.68)
 		(width 1)
 		(layer "B.Cu")
@@
 	)
 	(segment
-		(start 117.093056 106.68)
-		(end 136.652 106.68)
-		(width 1)
-		(layer "B.Cu")
-		(net 18)
-	)
-	(segment
 		(start 109.768 91.44)
 		(end 108.463 91.44)
@@
 	)
 	(segment
-		(start 108.463 91.44)
-		(end 108.209 91.186)
+		(start 109.768 98.846)
+		(end 117.602 106.68)
 		(width 1)
 		(layer "B.Cu")
@@
 	)
 	(segment
-		(start 109.768 91.44)
-		(end 114.046 95.718)
+		(start 108.463 91.44)
+		(end 108.209 91.186)
 		(width 1)
 		(layer "B.Cu")

Commit message: Added gerber
Routing:
- net Net-(R7-Pad2): track 43.4 -> 45.9 mm
- net Net-(Q1-B): track 157.2 -> 158.9 mm
- net Net-(U1A-+): track 53.7 -> 54.3 mm
- net IN: track 12.8 -> 12.3 mm
Changed lines of the file:
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@@
 		)
 		(pad "" np_thru_hole circle
-			(at -0.062 -0.008)
+			(at 0 0)
 			(size 2.2 2.2)
 			(drill 2.2)
@@
 	)
 	(segment
-		(start 103.632 77.002)
-		(end 101.723 75.093)
+		(start 173.255 54.672709)
+		(end 173.255 58.977)
 		(width 1)
 		(layer "B.Cu")
@@
 	)
 	(segment
-		(start 172.426 53.633)
-		(end 173.255 54.462)
+		(start 173.255 58.977)
+		(end 171.654 60.578)
 		(width 1)
 		(layer "B.Cu")
@@
 	)
 	(segment
-		(start 173.255 54.462)
-		(end 173.255 58.977)
-		(width 1)
-		(layer "B.Cu")
-		(net 3)
-	)
-	(segment
 		(start 108.209 78.486)
 		(end 105.116 78.486)
@@
 	)
 	(segment
-		(start 101.723 75.093)
-		(end 101.723 57.281)
+		(start 100.838 74.208)
+		(end 100.838 58.166)
 		(width 1)
 		(layer "B.Cu")
@@
 	)
 	(segment
-		(start 173.255 58.977)
-		(end 171.654 60.578)
+		(start 103.632 77.002)
+		(end 100.838 74.208)
 		(width 1)
 		(layer "B.Cu")
@@
 	)
 	(segment
-		(start 101.723 57.281)
-		(end 105.371 53.633)
+		(start 106.68 52.324)
+		(end 170.906291 52.324)
 		(width 1)
 		(layer "B.Cu")
@@
 	)
 	(segment
-		(start 105.371 53.633)
-		(end 172.426 53.633)
+		(start 100.838 58.166)
+		(end 106.68 52.324)
 		(width 1)
 		(layer "B.Cu")
@@
 	)
 	(segment
+		(start 170.906291 52.324)
+		(end 173.255 54.672709)
+		(width 1)
+		(layer "B.Cu")
+		(net 3)
+	)
+	(segment
 		(start 174.805 87.935944)
 		(end 173.666 86.796944)
@@
 	)
 	(segment
-		(start 103.124 64.262)
-		(end 103.124 58.166)
+		(start 121.666 55.285472)
+		(end 121.666 56.134)
 		(width 1)
 		(layer "B.Cu")
@@
 	)
 	(segment
-		(start 106.457 54.833)
-		(end 121.213528 54.833)
+		(start 120.482528 54.102)
+		(end 121.666 55.285472)
 		(width 1)
 		(layer "B.Cu")
@@
 	)
 	(segment
-		(start 121.666 59.984)
-		(end 122.642 60.96)
+		(start 107.188 54.102)
+		(end 120.482528 54.102)
 		(width 1)
 		(layer "B.Cu")
@@
 	)
 	(segment
-		(start 103.124 58.166)
-		(end 106.457 54.833)
+		(start 121.666 59.984)
+		(end 122.642 60.96)
 		(width 1)
 		(layer "B.Cu")
@@
 	)
 	(segment
-		(start 121.213528 54.833)
-		(end 121.666 55.285472)
+		(start 103.124 58.166)
+		(end 107.188 54.102)
 		(width 1)
 		(layer "B.Cu")
@@
 	)
 	(segment
-		(start 121.666 55.285472)
-		(end 121.666 56.134)
+		(start 103.124 64.262)
+		(end 103.124 58.166)
 		(width 1)
 		(layer "B.Cu")
@@
 	)
 	(segment
-		(start 111.506 56.134)
-		(end 110.716 56.924)
-		(width 1)
-		(layer "B.Cu")
-		(net 6)
-	)
-	(segment
 		(start 119.666 56.134)
-		(end 111.506 56.134)
-		(width 1)
-		(layer "B.Cu")
-		(net 6)
-	)
-	(segment
-		(start 111.506 56.134)
-		(end 111.0045 56.134)
+		(end 118.876 56.924)
 		(width 1)
 		(layer "B.Cu")
@@
 	)
 	(segment
-		(start 110.716 56.924)
+		(start 118.876 56.924)
 		(end 107.696 56.924)
 		(width 1)
@@
 	)
 	(segment
+		(start 148.59 87.376)
+		(end 148.59 84.836)
+		(width 1)
+		(layer "F.Cu")
+		(net 15)
+	)
+	(segment
 		(start 146.170944 87.376)
 		(end 142.303 83.508056)
@@
 	)
 	(segment
-		(start 138.470347 56.642)
-		(end 138.163347 56.335)
+		(start 146.558 56.642)
+		(end 146.251 56.335)
 		(width 4)
 		(layer "B.Cu")
@@
 	)
 	(segment
+		(start 146.251 56.335)
+		(end 136.398 56.335)
+		(width 4)
+		(layer "B.Cu")
+		(net 17)
+	)
+	(segment
 		(start 155.718651 70.258)
 		(end 147.32 61.859349)
@@
 	)
 	(segment
-		(start 138.163347 56.335)
-		(end 136.398 56.335)
-		(width 4)
-		(layer "B.Cu")
-		(net 17)
-	)
-	(segment
 		(start 132.958651 55.509349)
 		(end 136.398 55.509349)
@@
 		(layer "B.Cu")
 		(net 17)
-	)
-	(segment
-		(start 146.558 56.642)
-		(end 138.470347 56.642)
-		(width 4)
-		(layer "B.Cu")
-		(net 17)

Commit message: WIP
Routing:
- net B-: track 126.9 -> 124.7 mm
Changed lines of the file:
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@@
 			(outputformat 1)
 			(mirror no)
-			(drillshape 1)
+			(drillshape 0)
 			(scaleselection 1)
-			(outputdirectory "")
+			(outputdirectory "gerber")
 		)
 	)
@@
 	)
 	(segment
-		(start 145.288 102.77)
-		(end 158.496 89.562)
-		(width 4)
+		(start 171.654 58.298)
+		(end 170.053 59.899)
+		(width 1)
 		(layer "B.Cu")
 		(net 18)
 	)
 	(segment
-		(start 171.654 58.298)
-		(end 170.053 59.899)
-		(width 1)
+		(start 145.288 106.68)
+		(end 145.288 106.426)
+		(width 4)
 		(layer "B.Cu")
 		(net 18)
@@
 	)
 	(segment
+		(start 145.288 106.426)
+		(end 162.152 89.562)
+		(width 4)
+		(layer "B.Cu")
+		(net 18)
+	)
+	(segment
+		(start 169.284 89.562)
+		(end 170.654 90.932)
+		(width 4)
+		(layer "B.Cu")
+		(net 18)
+	)
+	(segment
 		(start 169.337791 83.531)
 		(end 167.48568 83.531)
@@
 	)
 	(segment
-		(start 145.288 106.68)
-		(end 145.288 102.77)
+		(start 162.152 89.562)
+		(end 169.284 89.562)
 		(width 4)
 		(layer "B.Cu")
@@
 	)
 	(segment
-		(start 169.284 89.562)
-		(end 170.654 90.932)
-		(width 4)
-		(layer "B.Cu")
-		(net 18)
-	)
-	(segment
 		(start 170.053 59.899)
 		(end 170.053 61.575)
@@
 		(layer "B.Cu")
 		(net 18)
-	)
-	(segment
-		(start 158.496 89.562)
-		(end 169.284 89.562)
-		(width 4)
-		(layer "B.Cu")
-		(net 18)

Commit message: WIP
Routing:
- net B-: track 124.7 -> 128.0 mm
Changed lines of the file:
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@@
 	)
 	(segment
-		(start 173.255 54.672709)
-		(end 173.255 58.977)
+		(start 169.672 52.324)
+		(end 171.196 53.848)
+		(width 1)
+		(layer "B.Cu")
+		(net 3)
+	)
+	(segment
+		(start 100.838 58.166)
+		(end 106.68 52.324)
+		(width 1)
+		(layer "B.Cu")
+		(net 3)
+	)
+	(segment
+		(start 106.68 52.324)
+		(end 169.672 52.324)
 		(width 1)
 		(layer "B.Cu")
@@
 	)
 	(segment
+		(start 173.255 53.848)
+		(end 173.255 58.977)
+		(width 1)
+		(layer "B.Cu")
+		(net 3)
+	)
+	(segment
+		(start 171.196 53.848)
+		(end 173.255 53.848)
+		(width 1)
+		(layer "B.Cu")
+		(net 3)
+	)
+	(segment
+		(start 174.805 79.760847)
+		(end 174.805 63.729)
+		(width 1)
+		(layer "B.Cu")
+		(net 3)
+	)
+	(segment
+		(start 171.654 107.326)
+		(end 173.464 107.326)
+		(width 1)
+		(layer "B.Cu")
+		(net 3)
+	)
+	(segment
+		(start 173.666 86.796944)
+		(end 173.666 80.899847)
+		(width 1)
+		(layer "B.Cu")
+		(net 3)
+	)
+	(segment
+		(start 108.209 78.486)
+		(end 105.116 78.486)
+		(width 1)
+		(layer "B.Cu")
+		(net 3)
+	)
+	(segment
+		(start 103.632 77.002)
+		(end 100.838 74.208)
+		(width 1)
+		(layer "B.Cu")
+		(net 3)
+	)
+	(segment
+		(start 105.116 78.486)
+		(end 103.632 77.002)
+		(width 1)
+		(layer "B.Cu")
+		(net 3)
+	)
+	(segment
+		(start 174.805 97.747847)
+		(end 174.805 87.935944)
+		(width 1)
+		(layer "B.Cu")
+		(net 3)
+	)
+	(segment
 		(start 173.255 58.977)
 		(end 171.654 60.578)
@@
 	)
 	(segment
-		(start 174.805 79.760847)
-		(end 174.805 63.729)
-		(width 1)
-		(layer "B.Cu")
-		(net 3)
-	)
-	(segment
-		(start 171.654 107.326)
-		(end 173.464 107.326)
-		(width 1)
-		(layer "B.Cu")
-		(net 3)
-	)
-	(segment
-		(start 173.666 86.796944)
-		(end 173.666 80.899847)
-		(width 1)
-		(layer "B.Cu")
-		(net 3)
-	)
-	(segment
-		(start 108.209 78.486)
-		(end 105.116 78.486)
-		(width 1)
-		(layer "B.Cu")
-		(net 3)
-	)
-	(segment
-		(start 105.116 78.486)
-		(end 103.632 77.002)
-		(width 1)
-		(layer "B.Cu")
-		(net 3)
-	)
-	(segment
 		(start 100.838 74.208)
 		(end 100.838 58.166)
@@
 	)
 	(segment
-		(start 174.805 97.747847)
-		(end 174.805 87.935944)
-		(width 1)
-		(layer "B.Cu")
-		(net 3)
-	)
-	(segment
-		(start 103.632 77.002)
-		(end 100.838 74.208)
-		(width 1)
-		(layer "B.Cu")
-		(net 3)
-	)
-	(segment
-		(start 106.68 52.324)
-		(end 170.906291 52.324)
-		(width 1)
-		(layer "B.Cu")
-		(net 3)
-	)
-	(segment
-		(start 100.838 58.166)
-		(end 106.68 52.324)
-		(width 1)
-		(layer "B.Cu")
-		(net 3)
-	)
-	(segment
 		(start 173.464 107.326)
 		(end 173.666 107.124)
@@
 	)
 	(segment
-		(start 170.906291 52.324)
-		(end 173.255 54.672709)
-		(width 1)
-		(layer "B.Cu")
-		(net 3)
-	)
-	(segment
 		(start 174.805 87.935944)
 		(end 173.666 86.796944)
@@
 	)
 	(segment
+		(start 157.48 94.234)
+		(end 162.152 89.562)
+		(width 4)
+		(layer "B.Cu")
+		(net 18)
+	)
+	(segment
 		(start 109.768 91.44)
 		(end 109.768 98.846)
@@
 	(segment
 		(start 145.288 106.426)
-		(end 162.152 89.562)
+		(end 157.48 94.234)
 		(width 4)
 		(layer "B.Cu")
@@
 	)
 	(segment
+		(start 157.48 94.234)
+		(end 156.718 94.234)
+		(width 4)
+		(layer "B.Cu")
+		(net 18)
+	)
+	(segment
 		(start 173.605 79.263791)
 		(end 169.337791 83.531)
@@
 		(layer "B.Cu")
 		(net 18)
+	)
+	(segment
+		(start 156.718 94.234)
+		(end 154.94 92.456)
+		(width 4)
+		(layer "B.Cu")
+		(net 18)
